File: REF-IN-BLE-NS 4-1.brd (EAGLE design)
At the start: 44 x 93.5 mm, 87 parts, among them U1 NRF52832_10QFN48, U2 AEM10941, X1 32 MHz, X2 32.768 kHz

Commit message: Update to v4-1
Changed filenames to reflect version change
fixes #1
Connections:
- net GND: now also U$7.P$4, U$7.P$5; no longer U$7.P$1
Routing:
- net GND: vias 64 -> 66
- added copper zone on layer 15, net GND
- added copper zone on layer 2, net GND
- added copper zone on layer 2, net N$33
- added copper zone on layer 15, net N$35
- added copper zone on layer 15, net N$39
Other:
- board text added: "BUTTON1"
- board text added: "LED3"
- board text added: "REF-IN-BLE-NS 4-1"
- board text added: "nRF Blinky"
- board text removed: "REF-IN-BLE-NS 4-0"
Changed lines of the file:
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@@
 <setting verticaltext="up"/>
 </settings>
-<grid distance="0.1" unitdist="mm" unit="mm" style="dots" multiple="1" display="yes" altdistance="0.003125" altunitdist="mic" altunit="mm"/>
+<grid distance="0.05" unitdist="mm" unit="mm" style="dots" multiple="1" display="yes" altdistance="0.003125" altunitdist="mic" altunit="mm"/>
 <layers>
 <layer number="1" name="Top" color="4" fill="1" visible="no" active="yes"/>
-<layer number="2" name="Route2" color="1" fill="3" visible="no" active="no"/>
+<layer number="2" name="Route2" color="1" fill="3" visible="no" active="yes"/>
 <layer number="3" name="Route3" color="4" fill="3" visible="no" active="no"/>
 <layer number="4" name="Route4" color="1" fill="4" visible="no" active="no"/>
@@
 <layer number="13" name="Route13" color="4" fill="5" visible="no" active="no"/>
 <layer number="14" name="Route14" color="1" fill="6" visible="no" active="no"/>
-<layer number="15" name="Route15" color="4" fill="6" visible="no" active="no"/>
+<layer number="15" name="Route15" color="4" fill="6" visible="no" active="yes"/>
 <layer number="16" name="Bottom" color="1" fill="1" visible="yes" active="yes"/>
 <layer number="17" name="Pads" color="2" fill="1" visible="yes" active="yes"/>
 <layer number="18" name="Vias" color="2" fill="1" visible="yes" active="yes"/>
 <layer number="19" name="Unrouted" color="6" fill="1" visible="no" active="yes"/>
-<layer number="20" name="Dimension" color="15" fill="1" visible="yes" active="yes"/>
+<layer number="20" name="Dimension" color="15" fill="1" visible="no" active="yes"/>
 <layer number="21" name="tPlace" color="7" fill="1" visible="no" active="yes"/>
 <layer number="22" name="bPlace" color="7" fill="1" visible="yes" active="yes"/>
-<layer number="23" name="tOrigins" color="15" fill="1" visible="no" active="yes"/>
+<layer number="23" name="tOrigins" color="15" fill="1" visible="yes" active="yes"/>
 <layer number="24" name="bOrigins" color="15" fill="1" visible="no" active="yes"/>
 <layer number="25" name="tNames" color="7" fill="1" visible="no" active="yes"/>
@@
 <board>
 <plain>
-<text x="1.9" y="56.765" size="0.85" layer="21" font="vector" ratio="10" rot="R90">REF-IN-BLE-NS 4-0</text>
-<text x="1.9" y="71.235" size="0.85" layer="21" font="vector" ratio="10" rot="R90">PowerFilm Solar</text>
+<text x="1.9" y="56.75" size="0.85" layer="21" font="vector" ratio="10" rot="R90">REF-IN-BLE-NS 4-1</text>
+<text x="1.9" y="71" size="0.85" layer="21" font="vector" ratio="10" rot="R90">PowerFilm Solar</text>
 <text x="28.4" y="11.1" size="1" layer="25" font="vector">U1</text>
 <wire x1="2.5" y1="22.5" x2="2.5" y2="7.5" width="0.3" layer="21" style="shortdash"/>
@@
 <text x="3.65" y="7.5" size="1.016" layer="22" font="vector" rot="MR0">CFG2</text>
 <text x="3.6" y="16" size="1.016" layer="22" font="vector" rot="MR0">CFG0</text>
-<text x="15.3" y="15.1" size="1.016" layer="22" font="vector" rot="MR90">ENHV</text>
+<text x="12.3" y="15.15" size="1.016" layer="22" font="vector" rot="MR90">ENHV</text>
 <text x="7.55" y="15.1" size="1.016" layer="22" font="vector" rot="MR90">ENLV</text>
 <text x="22.3" y="19.3" size="1.016" layer="22" font="vector" rot="R180">ENBAL</text>
@@
 <text x="21.2" y="23.6" size="1.016" layer="22" font="vector" rot="MR270">S1</text>
 <text x="18.6" y="23.6" size="1.016" layer="22" font="vector" rot="MR270">S0</text>
-<text x="1.2" y="5.6" size="0.85" layer="21" font="vector" ratio="10">REF-IN-BLE-NS 4-0</text>
+<text x="1.2" y="5.6" size="0.85" layer="21" font="vector" ratio="10">REF-IN-BLE-NS 4-1</text>
 <text x="1.2" y="3.8" size="0.85" layer="21" font="vector" ratio="10">PowerFilm Solar</text>
 <rectangle x1="13.1123" y1="35.1193" x2="14.7887" y2="35.132" layer="22" rot="R270"/>
@@
 <wire x1="31.5" y1="25.5" x2="12.5" y2="25.5" width="0" layer="20"/>
 <wire x1="12.5" y1="25.5" x2="12.5" y2="28" width="0" layer="20"/>
+<text x="18" y="6.9" size="0.8128" layer="21" font="vector">LED3</text>
+<text x="23.7" y="2.5" size="0.8128" layer="21" font="vector">BUTTON1</text>
+<text x="40.75" y="6.95" size="0.8128" layer="21" font="vector" rot="R90">nRF Blinky</text>
 </plain>
 <attributes>
@@
 Please make sure your boards conform to these design rules.
 &lt;/p&gt;</description>
-<param name="layerSetup" value="(1*16)"/>
+<param name="layerSetup" value="(1*2+15*16)"/>
 <param name="mtCopper" value="0.035559375mm 0.0356mm 0.0356mm 0.0356mm 0.0356mm 0.0356mm 0.0356mm 0.0356mm 0.0356mm 0.0356mm 0.0356mm 0.0356mm 0.0356mm 0.0356mm 0.0356mm 0.035559375mm"/>
 <param name="mtIsolate" value="1.6mm 0.1499mm 0.2007mm 0.1499mm 0.2007mm 0.1499mm 0.2007mm 0.1499mm 0.2007mm 0.1499mm 0.2007mm 0.1499mm 0.2007mm 0.1499mm 0.2007mm"/>
@@
 <contactref element="U2" pad="7"/>
 <contactref element="R9" pad="2"/>
-<contactref element="U$7" pad="P$1"/>
+<contactref element="U$7" pad="P$4"/>
 <contactref element="U$2" pad="IN0"/>
 <contactref element="U$4" pad="IN0"/>
@@
 <via x="16.1" y="12.75" extent="1-16" drill="0.3" diameter="0.6"/>
 <via x="23.55" y="20.5" extent="1-16" drill="0.3" diameter="0.6"/>
+<polygon width="0" layer="2" rank="2">
+<vertex x="0" y="0"/>
+<vertex x="37.35" y="0"/>
+<vertex x="37.35" y="25.45"/>
+<vertex x="44" y="25.5"/>
+<vertex x="44" y="93.5"/>
+<vertex x="0" y="93.5"/>
+</polygon>
+<polygon width="0" layer="15">
+<vertex x="0" y="0"/>
+<vertex x="37.35" y="0"/>
+<vertex x="37.35" y="25.5"/>
+<vertex x="44" y="25.5"/>
+<vertex x="44" y="93.5"/>
+<vertex x="0" y="93.5"/>
+</polygon>
+<contactref element="U$7" pad="P$5"/>
+<via x="34.8" y="15.3" extent="1-16" drill="0.3" diameter="0.6"/>
+<via x="29.4" y="18.05" extent="1-16" drill="0.3" diameter="0.6"/>
 </signal>
 <signal name="N$5">
@@
 </polygon>
 </signal>
+<signal name="N$33">
+<polygon width="0" layer="2" pour="cutout">
+<vertex x="8" y="25.5"/>
+<vertex x="12.5" y="25.5"/>
+<vertex x="12.5" y="28"/>
+<vertex x="8" y="28"/>
+</polygon>
+<polygon width="0" layer="2" pour="cutout">
+<vertex x="31.5" y="25.5"/>
+<vertex x="36" y="25.5"/>
+<vertex x="36" y="28"/>
+<vertex x="31.5" y="28"/>
+</polygon>
+</signal>
+<signal name="N$35">
+<polygon width="0" layer="15" pour="cutout">
+<vertex x="8" y="28"/>
+<vertex x="12.5" y="28"/>
+<vertex x="12.5" y="25.5"/>
+<vertex x="8" y="25.5"/>
+</polygon>
+</signal>
+<signal name="N$39">
+<polygon width="0" layer="15" pour="cutout">
+<vertex x="31.5" y="28"/>
+<vertex x="36" y="28"/>
+<vertex x="36" y="25.5"/>
+<vertex x="31.5" y="25.5"/>
+</polygon>
+</signal>

Commit message: v4-1 Final
Parts:
- removed U$34: DMG2302UK-13, 00_PF_Nordic:SOT-23-3-DIODESINC
- U$33: device 00-PF-DevKits:SOT-23-3-DIODESINC -> 00_PF_Nordic:SOT-23-3-DIODESINC
- U$7: value N/A -> DMG2302UK-13; device 00_PF_Nordic:SOLAR_CELL_37X54MM -> 00_PF_Nordic:SOT-23-3-DIODESINC
- moved U$7 51.9 mm to (16.1, 7.70), turned to 0 degrees
Connections:
- net GND: now also U$7.2; no longer U$34.3, U$7.P$4, U$7.P$5
- net N$29: no longer U$7.P$2, U$7.P$3
- net N$47: now also U$7.3; no longer U$34.2
- net STATUS0: now also U$7.1; no longer U$34.1
Routing:
- net N$40: track 0.00 -> 69.7 mm
- net N$47: track 6.77 -> 8.18 mm
- net GND: vias 66 -> 64
