File: REF-IN-BLE-NS 4-1.sch (EAGLE design)
At the start: 87 parts, among them U1 NRF52832_10QFN48, U2 AEM10941, X1 32 MHz, X2 32.768 kHz

Commit message: v4-1 Final
Parts:
- removed U$34: DMG2302UK-13, 00_PF_Nordic:DMG2302UK-13
- U$33: device 00-PF-DevKits:DMG2305U-13 -> 00_PF_Nordic:DMG2305U-13
- U$7: value N/A -> DMG2302UK-13; device 00_PF_Nordic:SOLAR_CELL -> 00_PF_Nordic:DMG2302UK-13
Connections:
- net GND: now also U$7.S; no longer U$34.S, U$7.GND
- net N$29: no longer U$7.VOUT
- net N$47: now also U$7.D; no longer U$34.D
- net STATUS0: now also U$7.G; no longer U$34.G
