File: Boards/Flex/REF-IN-BLE-NS 4-2.brd (EAGLE design)
At the start: 44 x 96.5 mm, 67 parts, among them U1 NRF52832_10QFN48, U2 AEM10941, X1 32 MHz, X2 32.768 kHz

Commit message: Removed internal pullups, changed xtal caps 12pf
Parts:
- C1, C17, C18, C2: value 9pF -> 12pF
Changed lines of the file:
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@@
 <elements>
 <element name="AE1" library="00_PF_Nordic" package="BLE_ANTENNA_NORDIC_FLIPPED" value="2.4GHZ_ANTENNAFLIPPED" x="37.375" y="13.3" smashed="yes" rot="R270"/>
-<element name="C1" library="resistor" package="C0603" value="9pF" x="35.2" y="19.81" smashed="yes" rot="R90">
+<element name="C1" library="resistor" package="C0603" value="12pF" x="35.2" y="19.81" smashed="yes" rot="R90">
 <attribute name="NAME" x="35.765" y="18.775" size="1" layer="25" font="vector" rot="R90"/>
 <attribute name="VALUE" value="12pF" x="37.105" y="19.175" size="1.27" layer="27" rot="R90"/>
@@
 <attribute name="MFG_PART#" value="CL10A105KP8NNNC " x="28.86" y="17.19" size="1.778" layer="27" rot="R90" display="off"/>
 </element>
-<element name="C2" library="resistor" package="C0603" value="9pF" x="32.9" y="19.8" smashed="yes">
+<element name="C2" library="resistor" package="C0603" value="12pF" x="32.9" y="19.8" smashed="yes">
 <attribute name="NAME" x="32.065" y="19.335" size="1" layer="25" font="vector"/>
 <attribute name="VALUE" value="12pF" x="32.265" y="17.895" size="1.27" layer="27"/>
@@
 <attribute name="MFG_PART#" value="" x="20.5" y="20.2" size="1.778" layer="28" rot="MR180" display="off"/>
 </element>
-<element name="C17" library="resistor" package="C0603" value="9pF" x="20.71" y="14.63" smashed="yes" rot="R90">
+<element name="C17" library="resistor" package="C0603" value="12pF" x="20.71" y="14.63" smashed="yes" rot="R90">
 <attribute name="PERCENTAGE" value="5%" x="20.71" y="14.63" size="1.778" layer="27" rot="R90" display="off"/>
 <attribute name="MFG_PART#" value="C0603C120J5GACTU" x="20.71" y="14.63" size="1.778" layer="27" rot="R90" display="off"/>
@@
 <attribute name="VALUE" x="22.615" y="13.995" size="0.7" layer="27" font="vector" rot="R90"/>
 </element>
-<element name="C18" library="resistor" package="C0603" value="9pF" x="20.69" y="11.42" smashed="yes" rot="R270">
+<element name="C18" library="resistor" package="C0603" value="12pF" x="20.69" y="11.42" smashed="yes" rot="R270">
 <attribute name="PERCENTAGE" value="5%" x="20.69" y="11.42" size="1.778" layer="27" rot="R270" display="off"/>
 <attribute name="MFG_PART#" value="C0603C120J5GACTU" x="20.69" y="11.42" size="1.778" layer="27" rot="R270" display="off"/>

Commit message: Finalized rigid & flex and code
Parts:
- removed U$23: N/A, 00_PF_Nordic:CAP-XX_A-TYPE
- removed U$24: N/A, 00_PF_Nordic:CAP-XX_S-TYPE
- removed U$25: N/A, 00_PF_Nordic:CAP-XX_W-TYPE
- removed U$26: N/A, 00_PF_Nordic:BZ01_L-TYPE
- removed U$27: N/A, 00_PF_Nordic:BZ059_N-TYPE
- removed U$28: N/A, 00_PF_Nordic:BZ01_S-TYPE
- removed U$29: N/A, 00_PF_Nordic:BZ05_S-TYPE
- removed U$30: N/A, 00_PF_Nordic:BZ09_S-TYPE
Connections:
- net BAL: no longer U$23.P$1, U$24.P$1, U$25.P$1, U$26.P$3, U$26.P$4, U$28.P$3, U$29.P$3, U$30.P$3
- net BATT: no longer U$23.P$2, U$24.P$2, U$25.P$2, U$26.P$1, U$26.P$2, U$27.P$1, U$28.P$1, U$28.P$2, U$29.P$1, U$29.P$2, U$30.P$1, U$30.P$2
- net GND: no longer U$23.P$3, U$24.P$3, U$25.P$3, U$27.P$2
Routing:
- net BATT: track 151.7 -> 40.2 mm
- net BAL: track 103.3 -> 26.6 mm
- net GND: track 49.6 -> 41.9 mm, vias 107 -> 104
Other:
- outline, holes or cut-outs redrawn
- board text removed: "+"
- board text removed: "-"
