File: Boards/Flex/REF-IN-BLE-NS 4-2.sch (EAGLE design)
At the start: 67 parts, among them U1 NRF52832_10QFN48, U2 AEM10941, X1 32 MHz, X2 32.768 kHz

Commit message: Removed internal pullups, changed xtal caps 12pf
Parts:
- C1, C17, C18, C2: value 9pF -> 12pF
Changed lines of the file:
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@@
 <parts>
 <part name="U1" library="00_PF_Nordic" deviceset="NRF52832_10QFN48" device=""/>
-<part name="C1" library="resistor" deviceset="C-US" device="C0603" technology="T-12PF" value="9pF"/>
+<part name="C1" library="resistor" deviceset="C-US" device="C0603" technology="T-12PF" value="12pF"/>
 <part name="L3" library="00_PF_Nordic" deviceset="L0603" device="" technology="V-15NH" value="15nH"/>
 <part name="L2" library="00_PF_Nordic" deviceset="L0603" device="" technology="V-10UH" value="10uH"/>
 <part name="L1" library="00_PF_Nordic" deviceset="L0603" device="" technology="V-3.9NH" value="3.9nH"/>
-<part name="C2" library="resistor" deviceset="C-US" device="C0603" technology="T-12PF" value="9pF"/>
+<part name="C2" library="resistor" deviceset="C-US" device="C0603" technology="T-12PF" value="12pF"/>
 <part name="C3" library="resistor" deviceset="C-US" device="C0603" technology="T-0.8PF" value="0.8pF"/>
 <part name="C4" library="resistor" deviceset="C-US" device="C0603" technology="T-100NF" value="100nF"/>
@@
 <part name="G19" library="supply2" deviceset="PE" device="" value="GND"/>
 <part name="U$11" library="00_PF_Nordic" deviceset="SOLDER_BRIGDE" device="CLOSED" value=""/>
-<part name="C17" library="resistor" deviceset="C-US" device="C0603" technology="T-12PF" value="9pF"/>
-<part name="C18" library="resistor" deviceset="C-US" device="C0603" technology="T-12PF" value="9pF"/>
+<part name="C17" library="resistor" deviceset="C-US" device="C0603" technology="T-12PF" value="12pF"/>
+<part name="C18" library="resistor" deviceset="C-US" device="C0603" technology="T-12PF" value="12pF"/>
 <part name="G20" library="supply2" deviceset="PE" device="" value="GND"/>
 <part name="X2" library="00_PF_Nordic" deviceset="FC-135_32.7680KA-AC" device="" value="32.768 kHz"/>

Commit message: Finalized rigid & flex and code
Parts:
- removed U$23: N/A, 00_PF_Nordic:CAP-XX_A-TYPE
- removed U$24: N/A, 00_PF_Nordic:CAP-XX_S-TYPE
- removed U$25: N/A, 00_PF_Nordic:CAP-XX_W-TYPE
- removed U$26: N/A, 00_PF_Nordic:BZ01_L-TYPE
- removed U$27: N/A, 00_PF_Nordic:BZ059_N-TYPE
- removed U$28: N/A, 00_PF_Nordic:BZ01_S-TYPE
- removed U$29: N/A, 00_PF_Nordic:BZ05_S-TYPE
- removed U$30: N/A, 00_PF_Nordic:BZ09_S-TYPE
Connections:
- net BAL: no longer U$23.BAL, U$24.BAL, U$25.BAL, U$26.2, U$28.2, U$29.2, U$30.2
- net BATT: no longer U$23.+, U$24.+, U$25.+, U$26.1, U$27.1, U$28.1, U$29.1, U$30.1
- net GND: no longer U$23.-, U$24.-, U$25.-, U$27.2
Other:
- note removed: "AVX Super-capacitors"
- note removed: "CAP-XX Super-capacitors"
- moved on the sheet: AE1, BUTTON1, C1, C10, C11, C17, C18, C2, C3, C4, C5, C6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
