File: Boards/Rigid/REF-IN-BLE-NS 4-2 Rigid.sch (EAGLE design)
At the start: 82 parts, among them U1 NRF52832_10QFN48, U2 AEM10941, X1 32 MHz, X2 32.768 kHz

Commit message: Removed internal pullups, changed xtal caps 12pf
Parts:
- C1, C17, C18, C2: value 9pF -> 12pF
Changed lines of the file:
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@@
 <parts>
 <part name="U1" library="00_PF_Nordic" deviceset="NRF52832_10QFN48" device=""/>
-<part name="C1" library="resistor" deviceset="C-US" device="C0603" technology="T-12PF" value="9pF"/>
+<part name="C1" library="resistor" deviceset="C-US" device="C0603" technology="T-12PF" value="12pF"/>
 <part name="L3" library="00_PF_Nordic" deviceset="L0603" device="" technology="V-15NH" value="15nH"/>
 <part name="L2" library="00_PF_Nordic" deviceset="L0603" device="" technology="V-10UH" value="10uH"/>
 <part name="L1" library="00_PF_Nordic" deviceset="L0603" device="" technology="V-3.9NH" value="3.9nH"/>
-<part name="C2" library="resistor" deviceset="C-US" device="C0603" technology="T-12PF" value="9pF"/>
+<part name="C2" library="resistor" deviceset="C-US" device="C0603" technology="T-12PF" value="12pF"/>
 <part name="C3" library="resistor" deviceset="C-US" device="C0603" technology="T-0.8PF" value="0.8pF"/>
 <part name="C4" library="resistor" deviceset="C-US" device="C0603" technology="T-100NF" value="100nF"/>
@@
 <part name="G19" library="supply2" deviceset="PE" device="" value="GND"/>
 <part name="U$11" library="00_PF_Nordic" deviceset="SOLDER_BRIGDE" device="CLOSED" value=""/>
-<part name="C17" library="resistor" deviceset="C-US" device="C0603" technology="T-12PF" value="9pF"/>
-<part name="C18" library="resistor" deviceset="C-US" device="C0603" technology="T-12PF" value="9pF"/>
+<part name="C17" library="resistor" deviceset="C-US" device="C0603" technology="T-12PF" value="12pF"/>
+<part name="C18" library="resistor" deviceset="C-US" device="C0603" technology="T-12PF" value="12pF"/>
 <part name="G20" library="supply2" deviceset="PE" device="" value="GND"/>
 <part name="X2" library="00_PF_Nordic" deviceset="FC-135_32.7680KA-AC" device="" value="32.768 kHz"/>

Commit message: Finalized rigid & flex and code
Parts:
- C17, C18: value 12pF -> 12p
- U$20: value 20PIN_CONN -> 18PIN_CONN; device 00_PF_Nordic:20PIN_CONN -> 00_PF_Nordic:18PIN_CONN
Connections:
- net GND: no longer U$20.P$20, U$20.P$9
- net P16: now also U$20.P$9; no longer U$20.P$19
Other:
- moved on the sheet: AE1, C1, C10, C11, C17, C18, C2, C3, C4, C5, C6, C7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
